File: Psion Keyboard.brd (EAGLE design)
At the start: 100 x 80 mm, 3 parts, among them X2 52745-2290

Commit message: Basic shape.
Parts:
- moved MS1 159.0 mm to (94.0, 22.9), turned to 180 degrees
- moved S2 53.3 mm to (33.0, 20.3), turned to 180 degrees
- moved X2 51.1 mm to (15.2, 17.8)
Changed lines of the file:
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@@
 </autorouter>
 <elements>
-<element name="MS1" library="adafruit" library_urn="urn:adsk.eagle:library:420" package="FEATHERWING_DIM" value="FEATHERWING_NODIM" x="-63.5" y="1.27"/>
-<element name="S2" library="adafruit" library_urn="urn:adsk.eagle:library:420" package="EG1213" value="EG1213" x="-19.05" y="31.75"/>
-<element name="X2" library="con-molex" library_urn="urn:adsk.eagle:library:165" package="52745-2290" value="52745-2290" x="-34.29" y="30.48">
-<attribute name="MF" value="MOLEX" x="-34.29" y="30.48" size="1.778" layer="27" display="off"/>
-<attribute name="MPN" value="" x="-34.29" y="30.48" size="1.778" layer="27" display="off"/>
-<attribute name="OC_FARNELL" value="unknown" x="-34.29" y="30.48" size="1.778" layer="27" display="off"/>
-<attribute name="OC_NEWARK" value="unknown" x="-34.29" y="30.48" size="1.778" layer="27" display="off"/>
+<element name="MS1" library="adafruit" library_urn="urn:adsk.eagle:library:420" package="FEATHERWING_DIM" value="FEATHERWING_NODIM" x="93.98" y="22.86" rot="R180"/>
+<element name="S2" library="adafruit" library_urn="urn:adsk.eagle:library:420" package="EG1213" value="EG1213" x="33.02" y="20.32" rot="R180"/>
+<element name="X2" library="con-molex" library_urn="urn:adsk.eagle:library:165" package="52745-2290" value="52745-2290" x="15.24" y="17.78">
+<attribute name="MF" value="MOLEX" x="15.24" y="17.78" size="1.778" layer="27" display="off"/>
+<attribute name="MPN" value="" x="15.24" y="17.78" size="1.778" layer="27" display="off"/>
+<attribute name="OC_FARNELL" value="unknown" x="15.24" y="17.78" size="1.778" layer="27" display="off"/>
+<attribute name="OC_NEWARK" value="unknown" x="15.24" y="17.78" size="1.778" layer="27" display="off"/>
 </element>
 </elements>
@@
 <contactref element="S2" pad="1"/>
 <contactref element="MS1" pad="4"/>
-<wire x1="-21.05" y1="31.75" x2="-49.53" y2="2.54" width="0" layer="19" extent="1-1"/>
+<wire x1="35.02" y1="20.32" x2="80.01" y2="21.59" width="0" layer="19" extent="1-1"/>
 </signal>
 <signal name="EN">
 <contactref element="S2" pad="2"/>
 <contactref element="MS1" pad="27"/>
-<wire x1="-19.05" y1="31.75" x2="-44.45" y2="22.86" width="0" layer="19" extent="1-1"/>
+<wire x1="33.02" y1="20.32" x2="74.93" y2="1.27" width="0" layer="19" extent="1-1"/>
 </signal>
 <signal name="SDA">
@@
 <contactref element="X2" pad="2"/>
 <contactref element="X2" pad="5"/>
-<wire x1="-37.54" y1="32.98" x2="-39.04" y2="32.98" width="0" layer="19" extent="1-1"/>
-<wire x1="-19.05" y1="22.86" x2="-37.54" y2="32.98" width="0" layer="19" extent="1-1"/>
+<wire x1="11.99" y1="20.28" x2="10.49" y2="20.28" width="0" layer="19" extent="1-1"/>
+<wire x1="49.53" y1="1.27" x2="11.99" y2="20.28" width="0" layer="19" extent="1-1"/>
 </signal>
 <signal name="SCL">
 <contactref element="MS1" pad="18"/>
 <contactref element="X2" pad="3"/>
-<wire x1="-21.59" y1="22.86" x2="-38.54" y2="32.98" width="0" layer="19" extent="1-1"/>
+<wire x1="52.07" y1="1.27" x2="10.99" y2="20.28" width="0" layer="19" extent="1-1"/>
 </signal>
 <signal name="27">
 <contactref element="MS1" pad="19"/>
 <contactref element="X2" pad="4"/>
-<wire x1="-24.13" y1="22.86" x2="-38.04" y2="32.98" width="0" layer="19" extent="1-1"/>
+<wire x1="54.61" y1="1.27" x2="11.49" y2="20.28" width="0" layer="19" extent="1-1"/>
 </signal>
 <signal name="30">
 <contactref element="MS1" pad="20"/>
 <contactref element="X2" pad="6"/>
-<wire x1="-26.67" y1="22.86" x2="-37.04" y2="32.98" width="0" layer="19" extent="1-1"/>
+<wire x1="57.15" y1="1.27" x2="12.49" y2="20.28" width="0" layer="19" extent="1-1"/>
 </signal>
 <signal name="11">
 <contactref element="MS1" pad="22"/>
 <contactref element="X2" pad="7"/>
-<wire x1="-36.54" y1="32.98" x2="-31.75" y2="22.86" width="0" layer="19" extent="1-1"/>
+<wire x1="12.99" y1="20.28" x2="62.23" y2="1.27" width="0" layer="19" extent="1-1"/>
 </signal>
 <signal name="7">
 <contactref element="MS1" pad="23"/>
 <contactref element="X2" pad="8"/>
-<wire x1="-36.04" y1="32.98" x2="-34.29" y2="22.86" width="0" layer="19" extent="1-1"/>
+<wire x1="13.49" y1="20.28" x2="64.77" y2="1.27" width="0" layer="19" extent="1-1"/>
 </signal>
 <signal name="15">
 <contactref element="MS1" pad="24"/>
 <contactref element="X2" pad="9"/>
-<wire x1="-35.54" y1="32.98" x2="-36.83" y2="22.86" width="0" layer="19" extent="1-1"/>
+<wire x1="13.99" y1="20.28" x2="67.31" y2="1.27" width="0" layer="19" extent="1-1"/>
 </signal>
 <signal name="16">
 <contactref element="MS1" pad="25"/>
 <contactref element="X2" pad="10"/>
-<wire x1="-35.04" y1="32.98" x2="-39.37" y2="22.86" width="0" layer="19" extent="1-1"/>
+<wire x1="14.49" y1="20.28" x2="69.85" y2="1.27" width="0" layer="19" extent="1-1"/>
 </signal>
 <signal name="USB">
@@
 <contactref element="MS1" pad="15"/>
 <contactref element="X2" pad="21"/>
-<wire x1="-29.54" y1="32.98" x2="-21.59" y2="2.54" width="0" layer="19" extent="1-1"/>
+<wire x1="19.99" y1="20.28" x2="52.07" y2="21.59" width="0" layer="19" extent="1-1"/>
 </signal>
 <signal name="RXD">
 <contactref element="MS1" pad="14"/>
 <contactref element="X2" pad="20"/>
-<wire x1="-30.04" y1="32.98" x2="-24.13" y2="2.54" width="0" layer="19" extent="1-1"/>
+<wire x1="19.49" y1="20.28" x2="54.61" y2="21.59" width="0" layer="19" extent="1-1"/>
 </signal>
 <signal name="MISO">
 <contactref element="MS1" pad="13"/>
 <contactref element="X2" pad="19"/>
-<wire x1="-30.54" y1="32.98" x2="-26.67" y2="2.54" width="0" layer="19" extent="1-1"/>
+<wire x1="18.99" y1="20.28" x2="57.15" y2="21.59" width="0" layer="19" extent="1-1"/>
 </signal>
 <signal name="MOSI">
 <contactref element="MS1" pad="12"/>
 <contactref element="X2" pad="18"/>
-<wire x1="-31.04" y1="32.98" x2="-29.21" y2="2.54" width="0" layer="19" extent="1-1"/>
+<wire x1="18.49" y1="20.28" x2="59.69" y2="21.59" width="0" layer="19" extent="1-1"/>
 </signal>
 <signal name="SCK">
 <contactref element="MS1" pad="11"/>
 <contactref element="X2" pad="17"/>
-<wire x1="-31.54" y1="32.98" x2="-31.75" y2="2.54" width="0" layer="19" extent="1-1"/>
+<wire x1="17.99" y1="20.28" x2="62.23" y2="21.59" width="0" layer="19" extent="1-1"/>
 </signal>
 <signal name="A5">
 <contactref element="MS1" pad="10"/>
 <contactref element="X2" pad="16"/>
-<wire x1="-32.04" y1="32.98" x2="-34.29" y2="2.54" width="0" layer="19" extent="1-1"/>
+<wire x1="17.49" y1="20.28" x2="64.77" y2="21.59" width="0" layer="19" extent="1-1"/>
 </signal>
 <signal name="A4">
 <contactref element="MS1" pad="9"/>
 <contactref element="X2" pad="15"/>
-<wire x1="-32.54" y1="32.98" x2="-36.83" y2="2.54" width="0" layer="19" extent="1-1"/>
+<wire x1="16.99" y1="20.28" x2="67.31" y2="21.59" width="0" layer="19" extent="1-1"/>
 </signal>
 <signal name="A3">
 <contactref element="MS1" pad="8"/>
 <contactref element="X2" pad="14"/>
-<wire x1="-33.04" y1="32.98" x2="-39.37" y2="2.54" width="0" layer="19" extent="1-1"/>
+<wire x1="16.49" y1="20.28" x2="69.85" y2="21.59" width="0" layer="19" extent="1-1"/>
 </signal>
 <signal name="A2">
 <contactref element="MS1" pad="7"/>
 <contactref element="X2" pad="13"/>
-<wire x1="-33.54" y1="32.98" x2="-41.91" y2="2.54" width="0" layer="19" extent="1-1"/>
+<wire x1="15.99" y1="20.28" x2="72.39" y2="21.59" width="0" layer="19" extent="1-1"/>
 </signal>
 <signal name="A1">
 <contactref element="MS1" pad="6"/>
 <contactref element="X2" pad="12"/>
-<wire x1="-34.04" y1="32.98" x2="-44.45" y2="2.54" width="0" layer="19" extent="1-1"/>
+<wire x1="15.49" y1="20.28" x2="74.93" y2="21.59" width="0" layer="19" extent="1-1"/>
 </signal>
 <signal name="A0">
 <contactref element="MS1" pad="5"/>
 <contactref element="X2" pad="11"/>
-<wire x1="-34.54" y1="32.98" x2="-46.99" y2="2.54" width="0" layer="19" extent="1-1"/>
+<wire x1="14.99" y1="20.28" x2="77.47" y2="21.59" width="0" layer="19" extent="1-1"/>
 </signal>
 </signals>
