File: pcb/psiboard.brd (EAGLE design)
At the start: 102.9 x 22.9 mm, 4 parts

Commit message: Schematic is now complete.
Connections:
- removed net N$1: KEYBOARD.2, KEYBOARD.5
- removed net N$26: KEYBOARD.3
- removed net N$27: KEYBOARD.4
- removed net N$29: KEYBOARD.6
- removed net N$30: KEYBOARD.7
- removed net N$31: KEYBOARD.8
- removed net N$32: KEYBOARD.9
- removed net N$33: KEYBOARD.10
- removed net N$34: KEYBOARD.11
- removed net N$35: KEYBOARD.12
- removed net N$36: KEYBOARD.13
- removed net N$37: KEYBOARD.14
- removed net N$38: KEYBOARD.15
- removed net N$39: KEYBOARD.16
- removed net N$40: KEYBOARD.17
- removed net N$41: KEYBOARD.18
- removed net N$42: KEYBOARD.19
- removed net N$43: KEYBOARD.20
- removed net N$44: KEYBOARD.21
- net 11: now also KEYBOARD.17
- net 12: now also KEYBOARD.7
- net 13: now also KEYBOARD.6
- net 14: now also KEYBOARD.4
- net 15: now also KEYBOARD.15
- net 16: now also KEYBOARD.14
- net 2: now also KEYBOARD.13
- net 25: now also KEYBOARD.21
- net 26: now also KEYBOARD.20
- net 27: now also KEYBOARD.19
- net 28: now also KEYBOARD.9
- net 29: now also KEYBOARD.8
- net 3: now also KEYBOARD.12
- net 30: now also KEYBOARD.18
- net 4: now also KEYBOARD.11
- net 5: now also KEYBOARD.10
- net 6: now also KEYBOARD.2, KEYBOARD.5
- net 7: now also KEYBOARD.16
- net 8: now also KEYBOARD.3
Other:
- board text added: "USB"
Changed lines of the file:
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@@
 <circle x="100.33" y="20.32" radius="1.27" width="0.1524" layer="20"/>
 <circle x="100.33" y="2.54" radius="1.27" width="0.1524" layer="20"/>
+<text x="40.005" y="13.97" size="1.4224" layer="21">USB</text>
 </plain>
 <attributes>
@@
 <signal name="25">
 <contactref element="FEATHER" pad="17"/>
+<contactref element="KEYBOARD" pad="21"/>
+<wire x1="17.45" y1="16.47" x2="58.42" y2="21.59" width="0" layer="19" extent="1-1"/>
 </signal>
 <signal name="26">
 <contactref element="FEATHER" pad="18"/>
+<contactref element="KEYBOARD" pad="20"/>
+<wire x1="16.95" y1="16.47" x2="60.96" y2="21.59" width="0" layer="19" extent="1-1"/>
 </signal>
 <signal name="27">
 <contactref element="FEATHER" pad="19"/>
+<contactref element="KEYBOARD" pad="19"/>
+<wire x1="16.45" y1="16.47" x2="63.5" y2="21.59" width="0" layer="19" extent="1-1"/>
 </signal>
 <signal name="30">
 <contactref element="FEATHER" pad="20"/>
+<contactref element="KEYBOARD" pad="18"/>
+<wire x1="15.95" y1="16.47" x2="66.04" y2="21.59" width="0" layer="19" extent="1-1"/>
 </signal>
 <signal name="11">
 <contactref element="FEATHER" pad="22"/>
+<contactref element="KEYBOARD" pad="17"/>
+<wire x1="15.45" y1="16.47" x2="71.12" y2="21.59" width="0" layer="19" extent="1-1"/>
 </signal>
 <signal name="7">
 <contactref element="FEATHER" pad="23"/>
+<contactref element="KEYBOARD" pad="16"/>
+<wire x1="14.95" y1="16.47" x2="73.66" y2="21.59" width="0" layer="19" extent="1-1"/>
 </signal>
 <signal name="15">
 <contactref element="FEATHER" pad="24"/>
+<contactref element="KEYBOARD" pad="15"/>
+<wire x1="14.45" y1="16.47" x2="76.2" y2="21.59" width="0" layer="19" extent="1-1"/>
 </signal>
 <signal name="16">
 <contactref element="FEATHER" pad="25"/>
+<contactref element="KEYBOARD" pad="14"/>
+<wire x1="13.95" y1="16.47" x2="78.74" y2="21.59" width="0" layer="19" extent="1-1"/>
 </signal>
 <signal name="USB">
@@
 <signal name="6">
 <contactref element="FEATHER" pad="15"/>
+<contactref element="KEYBOARD" pad="2"/>
+<contactref element="KEYBOARD" pad="5"/>
+<wire x1="9.45" y1="16.47" x2="60.96" y2="1.27" width="0" layer="19" extent="1-1"/>
+<wire x1="7.95" y1="16.47" x2="9.45" y2="16.47" width="0" layer="19" extent="1-1"/>
 </signal>
 <signal name="8">
 <contactref element="FEATHER" pad="14"/>
+<contactref element="KEYBOARD" pad="3"/>
+<wire x1="8.45" y1="16.47" x2="63.5" y2="1.27" width="0" layer="19" extent="1-1"/>
 </signal>
 <signal name="14">
 <contactref element="FEATHER" pad="13"/>
+<contactref element="KEYBOARD" pad="4"/>
+<wire x1="8.95" y1="16.47" x2="66.04" y2="1.27" width="0" layer="19" extent="1-1"/>
 </signal>
 <signal name="13">
 <contactref element="FEATHER" pad="12"/>
+<contactref element="KEYBOARD" pad="6"/>
+<wire x1="9.95" y1="16.47" x2="68.58" y2="1.27" width="0" layer="19" extent="1-1"/>
 </signal>
 <signal name="GND">
@@
 <signal name="2">
 <contactref element="FEATHER" pad="5"/>
+<contactref element="KEYBOARD" pad="13"/>
+<wire x1="13.45" y1="16.47" x2="86.36" y2="1.27" width="0" layer="19" extent="1-1"/>
 </signal>
 <signal name="3">
 <contactref element="FEATHER" pad="6"/>
+<contactref element="KEYBOARD" pad="12"/>
+<wire x1="12.95" y1="16.47" x2="83.82" y2="1.27" width="0" layer="19" extent="1-1"/>
 </signal>
 <signal name="4">
 <contactref element="FEATHER" pad="7"/>
+<contactref element="KEYBOARD" pad="11"/>
+<wire x1="12.45" y1="16.47" x2="81.28" y2="1.27" width="0" layer="19" extent="1-1"/>
 </signal>
 <signal name="5">
 <contactref element="FEATHER" pad="8"/>
+<contactref element="KEYBOARD" pad="10"/>
+<wire x1="11.95" y1="16.47" x2="78.74" y2="1.27" width="0" layer="19" extent="1-1"/>
 </signal>
 <signal name="28">
 <contactref element="FEATHER" pad="9"/>
+<contactref element="KEYBOARD" pad="9"/>
+<wire x1="11.45" y1="16.47" x2="76.2" y2="1.27" width="0" layer="19" extent="1-1"/>
 </signal>
 <signal name="29">
 <contactref element="FEATHER" pad="10"/>
+<contactref element="KEYBOARD" pad="8"/>
+<wire x1="10.95" y1="16.47" x2="73.66" y2="1.27" width="0" layer="19" extent="1-1"/>
 </signal>
 <signal name="12">
 <contactref element="FEATHER" pad="11"/>
-</signal>
-<signal name="N$26">
-<contactref element="KEYBOARD" pad="3"/>
-</signal>
-<signal name="N$27">
-<contactref element="KEYBOARD" pad="4"/>
-</signal>
-<signal name="N$29">
-<contactref element="KEYBOARD" pad="6"/>
-</signal>
-<signal name="N$30">
 <contactref element="KEYBOARD" pad="7"/>
-</signal>
-<signal name="N$31">
-<contactref element="KEYBOARD" pad="8"/>
-</signal>
-<signal name="N$32">
-<contactref element="KEYBOARD" pad="9"/>
-</signal>
-<signal name="N$33">
-<contactref element="KEYBOARD" pad="10"/>
-</signal>
-<signal name="N$34">
-<contactref element="KEYBOARD" pad="11"/>
-</signal>
-<signal name="N$35">
-<contactref element="KEYBOARD" pad="12"/>
-</signal>
-<signal name="N$36">
-<contactref element="KEYBOARD" pad="13"/>
-</signal>
-<signal name="N$37">
-<contactref element="KEYBOARD" pad="14"/>
-</signal>
-<signal name="N$38">
-<contactref element="KEYBOARD" pad="15"/>
-</signal>
-<signal name="N$39">
-<contactref element="KEYBOARD" pad="16"/>
-</signal>
-<signal name="N$40">
-<contactref element="KEYBOARD" pad="17"/>
-</signal>
-<signal name="N$41">
-<contactref element="KEYBOARD" pad="18"/>
-</signal>
-<signal name="N$42">
-<contactref element="KEYBOARD" pad="19"/>
-</signal>
-<signal name="N$43">
-<contactref element="KEYBOARD" pad="20"/>
-</signal>
-<signal name="N$44">
-<contactref element="KEYBOARD" pad="21"/>
+<wire x1="10.45" y1="16.47" x2="71.12" y2="1.27" width="0" layer="19" extent="1-1"/>
 </signal>
 <signal name="VBAT">
 <contactref element="FEATHER" pad="28"/>
 </signal>
-<signal name="N$1">
-<contactref element="KEYBOARD" pad="2"/>
-<contactref element="KEYBOARD" pad="5"/>
-<wire x1="9.45" y1="16.47" x2="7.95" y2="16.47" width="0" layer="19" extent="1-1"/>
-</signal>
 </signals>

Commit message: Routing complete.
Routing:
- net GND: track 0.00 -> 104.4 mm, vias 0 -> 1
- net 2: track 0.00 -> 80.1 mm
- net 3: track 0.00 -> 78.9 mm, vias 0 -> 2
- net 4: track 0.00 -> 75.7 mm
- net 5: track 0.00 -> 73.6 mm
- net 28: track 0.00 -> 73.3 mm, vias 0 -> 1
- net 16: track 0.00 -> 73.2 mm
- net 29: track 0.00 -> 69.3 mm
- net 15: track 0.00 -> 69.0 mm, vias 0 -> 1
- net 12: track 0.00 -> 68.1 mm, vias 0 -> 1
- net EN: track 0.00 -> 66.1 mm
- net 7: track 0.00 -> 65.4 mm
- net 13: track 0.00 -> 65.3 mm
- net 14: track 0.00 -> 63.7 mm
- net 6: track 0.00 -> 62.4 mm
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