File: pcb/psiboard.sch (EAGLE design)
At the start: 4 parts

Commit message: Schematic is now complete.
Connections:
- removed net N$1: KEYBOARD-2.S, KEYBOARD-5.S
- removed net N$26: KEYBOARD-3.S
- removed net N$27: KEYBOARD-4.S
- removed net N$29: KEYBOARD-6.S
- removed net N$30: KEYBOARD-7.S
- removed net N$31: KEYBOARD-8.S
- removed net N$32: KEYBOARD-9.S
- removed net N$33: KEYBOARD-10.S
- removed net N$34: KEYBOARD-11.S
- removed net N$35: KEYBOARD-12.S
- removed net N$36: KEYBOARD-13.S
- removed net N$37: KEYBOARD-14.S
- removed net N$38: KEYBOARD-15.S
- removed net N$39: KEYBOARD-16.S
- removed net N$40: KEYBOARD-17.S
- removed net N$41: KEYBOARD-18.S
- removed net N$42: KEYBOARD-19.S
- removed net N$43: KEYBOARD-20.S
- removed net N$44: KEYBOARD-21.S
- net 11: now also KEYBOARD-17.S
- net 12: now also KEYBOARD-7.S
- net 13: now also KEYBOARD-6.S
- net 14: now also KEYBOARD-4.S
- net 15: now also KEYBOARD-15.S
- net 16: now also KEYBOARD-14.S
- net 2: now also KEYBOARD-13.S
- net 25: now also KEYBOARD-21.S
- net 26: now also KEYBOARD-20.S
- net 27: now also KEYBOARD-19.S
- net 28: now also KEYBOARD-9.S
- net 29: now also KEYBOARD-8.S
- net 3: now also KEYBOARD-12.S
- net 30: now also KEYBOARD-18.S
- net 4: now also KEYBOARD-11.S
- net 5: now also KEYBOARD-10.S
- net 6: now also KEYBOARD-2.S, KEYBOARD-5.S
- net 7: now also KEYBOARD-16.S
- net 8: now also KEYBOARD-3.S

Commit message: Board design is generally working
Parts:
- removed U$1: MICRO-USB-B, micro usb B - 4LEGS:MICRO-USB-B
- added U$2: USB_MICRO_PWR, microB:USB_MICRO_PWR
Connections:
- removed net VBAT: FEATHER.VBAT
- net 11: now also KEYBOARD-7.S; no longer KEYBOARD-17.S
- net 12: now also KEYBOARD-17.S; no longer KEYBOARD-7.S
- net 13: now also KEYBOARD-18.S; no longer KEYBOARD-6.S
- net 14: now also KEYBOARD-19.S; no longer KEYBOARD-4.S
- net 15: now also KEYBOARD-9.S; no longer KEYBOARD-15.S
- net 16: now also KEYBOARD-10.S; no longer KEYBOARD-14.S
- net 2: now also KEYBOARD-11.S; no longer KEYBOARD-13.S
- net 25: now also KEYBOARD-2.S, KEYBOARD-5.S; no longer KEYBOARD-21.S
- net 26: now also KEYBOARD-3.S; no longer KEYBOARD-20.S
- net 27: now also KEYBOARD-4.S; no longer KEYBOARD-19.S
- net 28: now also KEYBOARD-15.S; no longer KEYBOARD-9.S
- net 29: now also KEYBOARD-16.S; no longer KEYBOARD-8.S
- net 30: now also KEYBOARD-6.S; no longer KEYBOARD-18.S
- net 4: now also KEYBOARD-13.S; no longer KEYBOARD-11.S
- net 5: now also KEYBOARD-14.S; no longer KEYBOARD-10.S
- net 6: now also KEYBOARD-21.S; no longer KEYBOARD-2.S, KEYBOARD-5.S
- net 7: now also KEYBOARD-8.S; no longer KEYBOARD-16.S
- net 8: now also KEYBOARD-20.S; no longer KEYBOARD-3.S
- net GND: now also U$2.GND; no longer U$1.GND
- net USB: now also U$2.VBUS; no longer U$1.VCC
